Commit message: added camera

File: sim_robot_description/urdf/robot_peripherals.xacro (robot description, xacro)
@@ -17,4 +17,5 @@
             </geometry>
         </collision>
+        <!-- NEED LIDAR INERTIA -->
     </link>
     <!-- lidar to chassis joint -->
@@ -24,3 +25,35 @@
         <child link = 'lidar_link'/>
     </joint>
+    <!-- camera link -->
+    <link name = 'camera_link'>
+        <visual>
+            <origin xyz = '0 0 0' rpy = '0 0 0'/>
+            <geometry>
+                <mesh filename = 'file://$(find sim_robot_description)/meshes/camera.STL'/>
+            </geometry>
+            <material name = 'black'/>
+        </visual>
+        <collision>
+            <origin xyz = '0 0 0' rpy = '0 0 0'/>
+            <geometry>
+                <mesh filename = 'file://$(find sim_robot_description)/meshes/camera.STL'/>
+            </geometry>
+        </collision>
+        <inertial>
+            <origin xyz = '0 0 0' rpy = '0 0 0'/>
+            <mass value = '0'/>
+            <inertia ixx = '0'
+                     ixy = '0'
+                     ixz = '0'
+                     iyy = '0'
+                     iyz = '0'
+                     izz = '0'/>
+        </inertial>
+    </link>
+    <!-- camera to chassis joint -->
+    <joint name = 'camera_joint' type = 'fixed'>
+        <origin xyz = '0.057105 1.7948E-05 0.03755' rpy = '0 0 0'/>
+        <parent link = 'chassis_link'/>
+        <child link = 'camera_link'/>
+    </joint>
 </robot>

Commit message: added lidar inertia and placed correctly

File: sim_robot_description/urdf/robot_peripherals.xacro (robot description, xacro)
@@ -5,21 +5,29 @@
     <link name = 'lidar_link'>
         <visual>
-            <origin xyz = '0 0 0' rpy = '0 0 0'/>
+            <origin xyz = '0 0 0' rpy = '1.570796 0 1.570796'/>
             <geometry>
-                <mesh filename = 'file://$(find sim_robot_description)/meshes/lidar.STL'/>
+                <mesh filename = 'file://$(find sim_robot_description)/meshes/lidar.STL' scale = '0.001 0.001 0.001'/>
             </geometry>
-            <material name = 'gray'/>
+            <material name = 'black'/>
         </visual>
         <collision>
-            <origin xyz = '0 0 0' rpy = '0 0 0'/>
+            <origin xyz = '0 0 0' rpy = '1.570796 0 1.570796'/>
             <geometry>
-                <mesh filename = 'file://$(find sim_robot_description)/meshes/lidar.STL'/>
+                <mesh filename = 'file://$(find sim_robot_description)/meshes/lidar.STL' scale = '0.001 0.001 0.001'/>
             </geometry>
         </collision>
-        <!-- NEED LIDAR INERTIA -->
+        <inertial>
+            <mass value = '0.19'/>
+            <inertia ixx = '1.244076063E-4'
+                     ixy = '0'
+                     ixz = '0'
+                     iyy = '1.244076063E-4'
+                     iyz = '0'
+                     izz = '2.0102E-4'/>
+        </inertial>
     </link>
     <!-- lidar to chassis joint -->
     <joint name = 'lidar_joint' type = 'fixed'>
-        <origin xyz = '0.0435 5.25826986680105E-05 0.11' rpy = '0 0 0'/>
+        <origin xyz = '0.0405 5.25826986680105E-05 0.08285' rpy = '0 0 0'/>
         <parent link = 'chassis_link'/>
         <child link = 'lidar_link'/>
@@ -41,5 +49,4 @@
         </collision>
         <inertial>
-            <origin xyz = '0 0 0' rpy = '0 0 0'/>
             <mass value = '0'/>
             <inertia ixx = '0'

Commit message: removed camera collision since it is inside of the main robot collision body

File: sim_robot_description/urdf/robot_peripherals.xacro (robot description, xacro)
@@ -42,10 +42,4 @@
             <material name = 'black'/>
         </visual>
-        <collision>
-            <origin xyz = '0 0 0' rpy = '0 0 0'/>
-            <geometry>
-                <mesh filename = 'file://$(find sim_robot_description)/meshes/camera.STL'/>
-            </geometry>
-        </collision>
         <inertial>
             <mass value = '0'/>

Commit message: approximated peripherals as simple geometries, added proper inertia to both, corrected camera mass

File: sim_robot_description/urdf/robot_peripherals.xacro (robot description, xacro)
@@ -12,17 +12,16 @@
         </visual>
         <collision>
-            <origin xyz = '0 0 0' rpy = '1.570796 0 1.570796'/>
+            <origin xyz = '0 0 -0.0005' rpy = '0 0 0'/>
             <geometry>
-                <mesh filename = 'file://$(find sim_robot_description)/meshes/lidar.STL' scale = '0.001 0.001 0.001'/>
+                <cylinder radius = '0.047' length = '0.04'/>
             </geometry>
         </collision>
         <inertial>
             <mass value = '0.19'/>
-            <inertia ixx = '1.244076063E-4'
-                     ixy = '0'
-                     ixz = '0'
-                     iyy = '1.244076063E-4'
-                     iyz = '0'
-                     izz = '2.0102E-4'/>
+            <xacro:cylinder_inertia
+                mass = '0.19'
+                radius = '0.047'
+                length = '0.04'
+            />
         </inertial>
     </link>
@@ -43,11 +42,11 @@
         </visual>
         <inertial>
-            <mass value = '0'/>
-            <inertia ixx = '0'
-                     ixy = '0'
-                     ixz = '0'
-                     iyy = '0'
-                     iyz = '0'
-                     izz = '0'/>
+            <mass value = '0.30393'/>
+            <xacro:box_inertia
+                mass = '0.30393'
+                w = '0.06'
+                h = '0.05'
+                d = '0.165'
+            />
         </inertial>
     </link>
