Commit message: added inertia macros and approximated all links as simple geometries with inertias based on this

File: sim_robot_description/urdf/robot_body_testing.xacro (robot description, xacro)
@@ -2,5 +2,5 @@
 <robot xmlns:xacro = 'http://www.ros.org/wiki/xacro'>
     <!-- PROPERTIES -->
-    <xacro:property name = 'a' value = '4'/>    <!--scalar used for inertia -->
+    <xacro:property name = 'a' value = '1'/>    <!--scalar used for inertia -->
     <xacro:property name = 'd' value = '0.5'/>  <!--scalar used for damping -->
     <material name = 'black'>
@@ -16,20 +16,20 @@
     <xacro:macro name = 'cylinder_inertia' params = 'mass radius length'>
         <inertia
-            ixx = '${mass * (3 * radius**2 + length**2) / 12}'
+            ixx = '${a * mass * (3 * radius**2 + length**2) / 12}'
             ixy = '0'
             ixz = '0'
-            iyy = '${mass * (3 * radius**2 + length**2) / 12}'
+            iyy = '${a * mass * (3 * radius**2 + length**2) / 12}'
             iyz = '0'
-            izz = '${mass * radius**2 / 12}'
+            izz = '${a * mass * radius**2 / 12}'
         />
     </xacro:macro>
     <xacro:macro name = 'box_inertia' params = 'mass w h d'>
         <inertia
-            ixx = '${mass * (h**2 + d**2) / 12}'
+            ixx = '${a * mass * (h**2 + d**2) / 12}'
             ixy = '0'
             ixz = '0'
-            iyy = '${mass * (w**2 + h**2) / 12}'
+            iyy = '${a * mass * (w**2 + h**2) / 12}'
             iyz = '0'
-            izz = '${mass * (w**2 + d**2) / 12}'
+            izz = '${a * mass * (w**2 + d**2) / 12}'
         />
     </xacro:macro>
@@ -67,5 +67,5 @@
         <parent link = 'base_link'/>
         <child link = 'chassis_link'/>
-        <origin xyz = '0 0 0.07115' rpy = '0 0 0'/>
+        <origin xyz = '0 0 0.07115' rpy = '0 0 0'/> <!-- origin offset of 0.07115 -->
     </joint>
     <!-- WHEEL LINKS & JOINTS -->
