Commit message: added ros2_control as a plugin. I do not like it

File: sim_robot_description/urdf/robot_gazebo_properties.xacro (robot description, xacro)
@@ -2,6 +2,6 @@
 <robot xmlns:xacro="http://www.ros.org/wiki/xacro">
     <!--            PROPERTIES          -->
-    <xacro:property name = 'mu1' value = '1.0'/>
-    <xacro:property name = 'mu2' value = '1.0'/>
+    <xacro:property name = 'mu1' value = '0.1'/>
+    <xacro:property name = 'mu2' value = '0.1'/>
     <!--            LINKS          -->
     <gazebo reference = 'chassis_link'>
@@ -31,8 +31,10 @@
         <material>Gazebo/Black</material>
     </gazebo>
-    <!--            GAZEBO CONTROL          -->
+    <gazebo reference = 'camera_link'>
+        <material>Gazebo/Black</material>
+    </gazebo>
+    <!--            GAZEBO CONTROL           -->
     <gazebo>
         <plugin name = 'omni_robot' filename = 'libgazebo_ros_omni_drive.so'>
-            <!-- setup -->
             <commandTopic>cmd_vel</commandTopic>
             <odometryTopic>odom</odometryTopic>
@@ -40,14 +42,11 @@
             <odometryRate>100.0</odometryRate>
             <robotBaseFrame>base_link</robotBaseFrame>
-            <!-- geometry -->
             <wheel_radius>0.03115</wheel_radius>
-            <base_length>0.162</base_length>
-            <base_width>0.17</base_width>
-            <!-- joints -->
+            <base_length>0.16</base_length>
+            <base_width>0.169</base_width>
             <front_left_joint>front_left_joint</front_left_joint>
             <front_right_joint>front_right_joint</front_right_joint>
             <rear_left_joint>back_left_joint</rear_left_joint>
             <rear_right_joint>back_right_joint</rear_right_joint>
-            <!-- config -->
             <wheel_max_speed>10.0</wheel_max_speed>
             <wheel_acceleration>10.0</wheel_acceleration>
@@ -55,3 +54,45 @@
         </plugin>
     </gazebo>
+    <!-- <ros2_control name = 'X3_Robot' type = 'system'>
+        <hardware>
+            <plugin>gazebo_ros2_control/GazeboSystem</plugin>
+        </hardware>
+        <joint name = 'front_left_joint'>
+            <command_interface name = 'velocity'>
+                <param name = 'min'> -1 </param>
+                <param name = 'max'> 1 </param>
+            </command_interface>
+            <state_interface name = 'velocity'/>
+            <state_interface name = 'position'/>
+        </joint>
+        <joint name = 'front_right_joint'>
+            <command_interface name = 'velocity'>
+                <param name = 'min'> -1 </param>
+                <param name = 'max'> 1 </param>
+            </command_interface>
+            <state_interface name = 'velocity'/>
+            <state_interface name = 'position'/>
+        </joint>
+        <joint name = 'back_left_joint'>
+            <command_interface name = 'velocity'>
+                <param name = 'min'> -1 </param>
+                <param name = 'max'> 1 </param>
+            </command_interface>
+            <state_interface name = 'velocity'/>
+            <state_interface name = 'position'/>
+        </joint>
+        <joint name = 'back_right_joint'>
+            <command_interface name = 'velocity'>
+                <param name = 'min'> -1 </param>
+                <param name = 'max'> 1 </param>
+            </command_interface>
+            <state_interface name = 'velocity'/>
+            <state_interface name = 'position'/>
+        </joint>
+    </ros2_control>
+    <gazebo>
+        <plugin filename = 'libgazebo_ros2_control.so' name = 'gazebo_ros2_control'>
+            <parameters>$(find sim_robot_description)/config/my_controllers.yaml</parameters>
+        </plugin>
+    </gazebo> -->
 </robot>

Commit message: removed ros2_control, added minDepth, kp, and kd as per https://robotics.stackexchange.com/questions/28808/the-robot-is-rotating-by-iteself-without-any-forces-or-input-why-and-how-can-i

File: sim_robot_description/urdf/robot_gazebo_properties.xacro (robot description, xacro)
@@ -2,6 +2,6 @@
 <robot xmlns:xacro="http://www.ros.org/wiki/xacro">
     <!--            PROPERTIES          -->
-    <xacro:property name = 'mu1' value = '0.1'/>
-    <xacro:property name = 'mu2' value = '0.1'/>
+    <xacro:property name = 'mu1' value = '0.7'/>
+    <xacro:property name = 'mu2' value = '0.7'/>
     <!--            LINKS          -->
     <gazebo reference = 'chassis_link'>
@@ -12,4 +12,7 @@
         <mu1 value = '${mu1}' />
         <mu2 value = '${mu2}' />
+        <minDepth>0.0001</minDepth>
+        <kp>100000</kp>
+        <kd>2500</kd>
     </gazebo>
     <gazebo reference = 'front_left_wheel_link'>
@@ -17,4 +20,7 @@
         <mu1 value = '${mu1}' />
         <mu2 value = '${mu2}' />
+        <minDepth>0.0001</minDepth>
+        <kp>100000</kp>
+        <kd>2500</kd>
     </gazebo>
     <gazebo reference = 'back_right_wheel_link'>
@@ -22,4 +28,7 @@
         <mu1 value = '${mu1}' />
         <mu2 value = '${mu2}' />
+        <minDepth>0.0001</minDepth>
+        <kp>100000</kp>
+        <kd>2500</kd>
     </gazebo>
     <gazebo reference = 'back_left_wheel_link'>
@@ -27,4 +36,7 @@
         <mu1 value = '${mu1}' />
         <mu2 value = '${mu2}' />
+        <minDepth>0.0001</minDepth>
+        <kp>100000</kp>
+        <kd>2500</kd>
     </gazebo>
     <gazebo reference = 'lidar_link'>
@@ -42,57 +54,15 @@
             <odometryRate>100.0</odometryRate>
             <robotBaseFrame>base_link</robotBaseFrame>
-            <wheel_radius>0.03115</wheel_radius>
+            <wheel_radius>0.0325</wheel_radius>
             <base_length>0.16</base_length>
             <base_width>0.169</base_width>
+            <front_right_joint>front_right_joint</front_right_joint>
             <front_left_joint>front_left_joint</front_left_joint>
-            <front_right_joint>front_right_joint</front_right_joint>
+            <rear_right_joint>back_right_joint</rear_right_joint>
             <rear_left_joint>back_left_joint</rear_left_joint>
-            <rear_right_joint>back_right_joint</rear_right_joint>
-            <wheel_max_speed>10.0</wheel_max_speed>
-            <wheel_acceleration>10.0</wheel_acceleration>
+            <wheel_max_speed>5.0</wheel_max_speed>
+            <wheel_acceleration>5.0</wheel_acceleration>
             <joint_config>1 1 1 1</joint_config>
         </plugin>
     </gazebo>
-    <!-- <ros2_control name = 'X3_Robot' type = 'system'>
-        <hardware>
-            <plugin>gazebo_ros2_control/GazeboSystem</plugin>
-        </hardware>
-        <joint name = 'front_left_joint'>
-            <command_interface name = 'velocity'>
-                <param name = 'min'> -1 </param>
-                <param name = 'max'> 1 </param>
-            </command_interface>
-            <state_interface name = 'velocity'/>
-            <state_interface name = 'position'/>
-        </joint>
-        <joint name = 'front_right_joint'>
-            <command_interface name = 'velocity'>
-                <param name = 'min'> -1 </param>
-                <param name = 'max'> 1 </param>
-            </command_interface>
-            <state_interface name = 'velocity'/>
-            <state_interface name = 'position'/>
-        </joint>
-        <joint name = 'back_left_joint'>
-            <command_interface name = 'velocity'>
-                <param name = 'min'> -1 </param>
-                <param name = 'max'> 1 </param>
-            </command_interface>
-            <state_interface name = 'velocity'/>
-            <state_interface name = 'position'/>
-        </joint>
-        <joint name = 'back_right_joint'>
-            <command_interface name = 'velocity'>
-                <param name = 'min'> -1 </param>
-                <param name = 'max'> 1 </param>
-            </command_interface>
-            <state_interface name = 'velocity'/>
-            <state_interface name = 'position'/>
-        </joint>
-    </ros2_control>
-    <gazebo>
-        <plugin filename = 'libgazebo_ros2_control.so' name = 'gazebo_ros2_control'>
-            <parameters>$(find sim_robot_description)/config/my_controllers.yaml</parameters>
-        </plugin>
-    </gazebo> -->
 </robot>

Commit message: added fdir1 tags

File: sim_robot_description/urdf/robot_gazebo_properties.xacro (robot description, xacro)
@@ -1,4 +1,4 @@
 <?xml version="1.0"?>
-<robot xmlns:xacro="http://www.ros.org/wiki/xacro">
+<robot xmlns:xacro="http://www.ros.org/wiki/xacro" xmlns:gz="http://gazebosim.org/schema">
     <!--            PROPERTIES          -->
     <xacro:property name = 'mu1' value = '1.5'/>
@@ -9,34 +9,38 @@
     </gazebo>
     <gazebo reference = 'front_right_wheel_link'>
-        <material>Gazebo/Black</material>
+        <material>Gazebo/Blue</material>
         <mu1 value = '${mu1}' />
         <mu2 value = '${mu2}' />
-        <minDepth>0.001</minDepth>
-        <kp>500000</kp>
-        <kd>1</kd>
+        <fdir1 gz:expressed_in='base_link'>1 1 0</fdir1>
+        <minDepth>0.0005</minDepth>
+        <kp>1000000</kp>
+        <kd>7500</kd>
     </gazebo>
     <gazebo reference = 'front_left_wheel_link'>
-        <material>Gazebo/Black</material>
+        <material>Gazebo/Blue</material>
         <mu1 value = '${mu1}' />
         <mu2 value = '${mu2}' />
-        <minDepth>0.001</minDepth>
-        <kp>500000</kp>
-        <kd>1</kd>
+        <fdir1 gz:expressed_in='base_link'>1 -1 0</fdir1>
+        <minDepth>0.0005</minDepth>
+        <kp>1000000</kp>
+        <kd>7500</kd>
     </gazebo>
     <gazebo reference = 'back_right_wheel_link'>
-        <material>Gazebo/Black</material>
+        <material>Gazebo/Blue</material>
         <mu1 value = '${mu1}' />
         <mu2 value = '${mu2}' />
-        <minDepth>0.001</minDepth>
-        <kp>500000</kp>
-        <kd>1</kd>
+        <fdir1 gz:expressed_in='base_link'>1 -1 0</fdir1>
+        <minDepth>0.0005</minDepth>
+        <kp>1000000</kp>
+        <kd>7500</kd>
     </gazebo>
     <gazebo reference = 'back_left_wheel_link'>
-        <material>Gazebo/Black</material>
+        <material>Gazebo/Blue</material>
         <mu1 value = '${mu1}' />
         <mu2 value = '${mu2}' />
-        <minDepth>0.001</minDepth>
-        <kp>500000</kp>
-        <kd>1</kd>
+        <fdir1 gz:expressed_in='base_link'>1 1 0</fdir1>
+        <minDepth>0.0005</minDepth>
+        <kp>1000000</kp>
+        <kd>7500</kd>
     </gazebo>
     <gazebo reference = 'lidar_link'>
@@ -52,5 +56,5 @@
             <odometryTopic>odom</odometryTopic>
             <odometryFrame>odom</odometryFrame>
-            <odometryRate>100.0</odometryRate>
+            <odometryRate>250.0</odometryRate>
             <robotBaseFrame>base_link</robotBaseFrame>
             <wheel_radius>0.0325</wheel_radius>
@@ -62,5 +66,5 @@
             <rear_left_joint>back_left_joint</rear_left_joint>
             <wheel_max_speed>10.0</wheel_max_speed>
-            <wheel_acceleration>10.0</wheel_acceleration>
+            <wheel_acceleration>15.0</wheel_acceleration>
             <joint_config>1 1 1 1</joint_config>
         </plugin>

Commit message: added physics engine macros

File: sim_robot_description/urdf/robot_gazebo_properties.xacro (robot description, xacro)
@@ -4,4 +4,7 @@
     <xacro:property name = 'mu1' value = '1.5'/>
     <xacro:property name = 'mu2' value = '0.05'/>
+    <xacro:property name = 'minDepth' value = '0.0005'/>
+    <xacro:property name = 'kp' value = '1000000'/>
+    <xacro:property name = 'kd' value = '7500'/>
     <!--            LINKS          -->
     <gazebo reference = 'chassis_link'>
@@ -9,38 +12,38 @@
     </gazebo>
     <gazebo reference = 'front_right_wheel_link'>
-        <material>Gazebo/Blue</material>
+        <material>Gazebo/Black</material>
         <mu1 value = '${mu1}' />
         <mu2 value = '${mu2}' />
         <fdir1 gz:expressed_in='base_link'>1 1 0</fdir1>
-        <minDepth>0.0005</minDepth>
-        <kp>1000000</kp>
-        <kd>7500</kd>
+        <minDepth>${minDepth}</minDepth>
+        <kp>${kp}</kp>
+        <kd>${kd}</kd>
     </gazebo>
     <gazebo reference = 'front_left_wheel_link'>
-        <material>Gazebo/Blue</material>
+        <material>Gazebo/Black</material>
         <mu1 value = '${mu1}' />
         <mu2 value = '${mu2}' />
         <fdir1 gz:expressed_in='base_link'>1 -1 0</fdir1>
-        <minDepth>0.0005</minDepth>
-        <kp>1000000</kp>
-        <kd>7500</kd>
+        <minDepth>${minDepth}</minDepth>
+        <kp>${kp}</kp>
+        <kd>${kd}</kd>
     </gazebo>
     <gazebo reference = 'back_right_wheel_link'>
-        <material>Gazebo/Blue</material>
+        <material>Gazebo/Black</material>
         <mu1 value = '${mu1}' />
         <mu2 value = '${mu2}' />
         <fdir1 gz:expressed_in='base_link'>1 -1 0</fdir1>
-        <minDepth>0.0005</minDepth>
-        <kp>1000000</kp>
-        <kd>7500</kd>
+        <minDepth>${minDepth}</minDepth>
+        <kp>${kp}</kp>
+        <kd>${kd}</kd>
     </gazebo>
     <gazebo reference = 'back_left_wheel_link'>
-        <material>Gazebo/Blue</material>
+        <material>Gazebo/Black</material>
         <mu1 value = '${mu1}' />
         <mu2 value = '${mu2}' />
         <fdir1 gz:expressed_in='base_link'>1 1 0</fdir1>
-        <minDepth>0.0005</minDepth>
-        <kp>1000000</kp>
-        <kd>7500</kd>
+        <minDepth>${minDepth}</minDepth>
+        <kp>${kp}</kp>
+        <kd>${kd}</kd>
     </gazebo>
     <gazebo reference = 'lidar_link'>

Commit message: HOLONOMIC BAY-BEE

File: sim_robot_description/urdf/robot_gazebo_properties.xacro (robot description, xacro)
@@ -2,7 +2,7 @@
 <robot xmlns:xacro="http://www.ros.org/wiki/xacro" xmlns:gz="http://gazebosim.org/schema">
     <!--            PROPERTIES          -->
-    <xacro:property name = 'mu1' value = '1.5'/>
-    <xacro:property name = 'mu2' value = '0.05'/>
-    <xacro:property name = 'minDepth' value = '0.0005'/>
+    <xacro:property name = 'mu1' value = '0.25'/>
+    <xacro:property name = 'mu2' value = '0.0'/>
+    <xacro:property name = 'minDepth' value = '0.0001'/>
     <xacro:property name = 'kp' value = '1000000'/>
     <xacro:property name = 'kd' value = '7500'/>
@@ -24,5 +24,5 @@
         <mu1 value = '${mu1}' />
         <mu2 value = '${mu2}' />
-        <fdir1 gz:expressed_in='base_link'>1 -1 0</fdir1>
+        <fdir1 gz:expressed_in='base_link'>-1 1 0</fdir1>
         <minDepth>${minDepth}</minDepth>
         <kp>${kp}</kp>
@@ -42,5 +42,5 @@
         <mu1 value = '${mu1}' />
         <mu2 value = '${mu2}' />
-        <fdir1 gz:expressed_in='base_link'>1 1 0</fdir1>
+        <fdir1 gz:expressed_in='base_link'>-1 -1 0</fdir1>
         <minDepth>${minDepth}</minDepth>
         <kp>${kp}</kp>
@@ -68,6 +68,6 @@
             <rear_right_joint>back_right_joint</rear_right_joint>
             <rear_left_joint>back_left_joint</rear_left_joint>
-            <wheel_max_speed>10.0</wheel_max_speed>
-            <wheel_acceleration>15.0</wheel_acceleration>
+            <wheel_max_speed>7.50</wheel_max_speed>
+            <wheel_acceleration>7.50</wheel_acceleration>
             <joint_config>1 1 1 1</joint_config>
         </plugin>

Commit message: added the lidar parameters

File: sim_robot_description/urdf/robot_gazebo_properties.xacro (robot description, xacro)
@@ -2,6 +2,6 @@
 <robot xmlns:xacro="http://www.ros.org/wiki/xacro" xmlns:gz="http://gazebosim.org/schema">
     <!--            PROPERTIES          -->
-    <xacro:property name = 'mu1' value = '0.25'/>
-    <xacro:property name = 'mu2' value = '0.0'/>
+    <xacro:property name = 'mu1' value = '0.1'/>
+    <xacro:property name = 'mu2' value = '0.1'/>
     <xacro:property name = 'minDepth' value = '0.0001'/>
     <xacro:property name = 'kp' value = '1000000'/>
@@ -49,4 +49,30 @@
     <gazebo reference = 'lidar_link'>
         <material>Gazebo/Black</material>
+        <sensor name = 'lidar' type = 'ray'>
+            <pose> 0 0 0 0 0 0 </pose>
+            <visualize>false</visualize>
+            <update_rate>10</update_rate>
+            <ray>
+                <scan>
+                    <horizontal>
+                        <samples>3200</samples>         <!-- 360 degrees divided by 0.1125 degree resolution -->
+                        <resolution>1</resolution>
+                        <min_angle>-3.14</min_angle>
+                        <max_angle>3.14</max_angle>
+                    </horizontal>
+                </scan>
+                <range>
+                    <min>0.05</min>
+                    <max>30.0</max>
+                </range>
+            </ray>
+            <plugin name = 'laser_controller' filename = 'libgazebo_ros_ray_sensor.so'>
+                <ros>
+                    <argument>~/out:=scan</argument>
+                </ros>
+                <output_type>sensor_msgs/LaserScan</output_type>
+                <frame_name>lidar_link</frame_name>
+            </plugin>
+        </sensor>
     </gazebo>
     <gazebo reference = 'camera_link'>

Commit message: added depth camera

File: sim_robot_description/urdf/robot_gazebo_properties.xacro (robot description, xacro)
@@ -5,5 +5,5 @@
     <xacro:property name = 'mu2' value = '0.1'/>
     <xacro:property name = 'minDepth' value = '0.0001'/>
-    <xacro:property name = 'kp' value = '1000000'/>
+    <xacro:property name = 'kp' value = '1e8'/>
     <xacro:property name = 'kd' value = '7500'/>
     <!--            LINKS          -->
@@ -13,4 +13,5 @@
     <gazebo reference = 'front_right_wheel_link'>
         <material>Gazebo/Black</material>
+        <pose>0 0 0 0 0 0</pose>
         <mu1 value = '${mu1}' />
         <mu2 value = '${mu2}' />
@@ -22,4 +23,5 @@
     <gazebo reference = 'front_left_wheel_link'>
         <material>Gazebo/Black</material>
+        <pose>0 0 0 0 0 0</pose>
         <mu1 value = '${mu1}' />
         <mu2 value = '${mu2}' />
@@ -31,4 +33,5 @@
     <gazebo reference = 'back_right_wheel_link'>
         <material>Gazebo/Black</material>
+        <pose>0 0 0 0 0 0</pose>
         <mu1 value = '${mu1}' />
         <mu2 value = '${mu2}' />
@@ -40,4 +43,5 @@
     <gazebo reference = 'back_left_wheel_link'>
         <material>Gazebo/Black</material>
+        <pose>0 0 0 0 0 0</pose>
         <mu1 value = '${mu1}' />
         <mu2 value = '${mu2}' />
@@ -51,5 +55,5 @@
         <sensor name = 'lidar' type = 'ray'>
             <pose> 0 0 0 0 0 0 </pose>
-            <visualize>true</visualize>
+            <visualize>false</visualize>
             <update_rate>10</update_rate>
             <ray>
@@ -78,4 +82,25 @@
     <gazebo reference = 'camera_link'>
         <material>Gazebo/Black</material>
+        <sensor name = 'camera' type = 'depth'>
+            <pose> 0 0 0 0 0 0 </pose>
+            <visualize>true</visualize>
+            <update_rate>10</update_rate>
+            <camera>
+                <horizontal_fov>1.019272283</horizontal_fov>
+                <vertical_fov>0.7941248097</vertical_fov>
+                <image>
+                    <format>R16G16B16</format>
+                    <width>640</width>
+                    <height>480</height>
+                </image>
+                <clip>
+                    <near>0.6</near>
+                    <far>8.0</far>
+                </clip>
+            </camera>
+            <plugin name = 'camera_controller' filename = 'libgazebo_ros_camera.so'>
+                <frame_name>camera_link_optical</frame_name>
+            </plugin>
+        </sensor>
     </gazebo>
     <!--            GAZEBO CONTROL           -->
@@ -86,5 +111,5 @@
             <odometryFrame>odom</odometryFrame>
             <odometryRate>250.0</odometryRate>
-            <robotBaseFrame>base_link</robotBaseFrame>
+            <robotBaseFrame>base_footprint</robotBaseFrame>
             <wheel_radius>0.0325</wheel_radius>
             <base_length>0.16</base_length>

File: sim_robot_description/urdf/robot_peripherals.xacro (robot description, xacro)
@@ -57,3 +57,12 @@
         <child link = 'camera_link'/>
     </joint>
+    <!-- optical link for camera coordinate frame -->
+    <link name = 'camera_link_optical'>
+    </link>
+    <!-- optical camera link to actual camera link joint: -->
+    <joint name = 'camera_optical_joint' type = 'fixed'>
+        <origin xyz = '0 0 0' rpy = '-1.570796 0 -1.570796'/>
+        <parent link = 'camera_link'/>
+        <child link = 'camera_link_optical'/>
+    </joint>
 </robot>
