Commit message: added IMU link

File: sim_robot_description/urdf/robot_body.xacro (robot description, xacro)
@@ -11,4 +11,7 @@
     <!-- base link -->
     <link name = 'base_link'>
+    </link>
+    <!-- imu link -->
+    <link name = 'imu_link'>
     </link>
     <!-- chassis link -->
@@ -27,4 +30,16 @@
             </geometry>
         </collision>
+        <inertial>
+            <origin xyz="0.00498197982182523 5.70233829969297E-05 -0.0121008098068578" rpy="0 0 0"/>
+            <!-- <mass value="0.486218814966626"/> -->
+            <mass value="2.415"/> <!--corrected mass value measured w/o wheels-->
+            <inertia
+                    ixx="${a*0.00196277727666921}"
+                    ixy="${a*2.50447049446755E-07}"
+                    ixz="${a*0.000140534767811098}"
+                    iyy="${a*0.00457256033711368}"
+                    iyz="${a*2.68618064993882E-07}"
+                    izz="${a*0.00493927269870476}"/>
+        </inertial>
     </link>
     <!-- chassis to base link joint -->
@@ -34,3 +49,9 @@
         <origin xyz = '0.0 0.0 0.07115' rpy = '0 0 0'/>
     </joint>
+    <!-- imu to chassis joint -->
+    <joint name="base_imu" type="fixed">
+        <parent link="chassis_link"/>
+        <child link="imu_link"/>
+        <origin xyz="-0.06 0.01 0.01" rpy="0 3.1415 1.5707"/>
+    </joint>
 </robot>

Commit message: added the four wheels

File: sim_robot_description/urdf/robot_body.xacro (robot description, xacro)
@@ -1,5 +1,5 @@
-<?xml version="1.0"?>
-<robot xmlns:xacro="http://www.ros.org/wiki/xacro">
-    <!-- properties -->
+<?xml version = '1.0'?>
+<robot xmlns:xacro = 'http://www.ros.org/wiki/xacro'>
+    <!-- PROPERTIES -->
     <xacro:property name='a' value='4'/>
     <material name = 'black'>
@@ -9,4 +9,5 @@
         <color rgba = '0 0.7 0 1'/>
     </material>
+    <!-- BASE LINK & JOINTS-->
     <!-- base link -->
     <link name = 'base_link'>
@@ -31,14 +32,13 @@
         </collision>
         <inertial>
-            <origin xyz="0.00498197982182523 5.70233829969297E-05 -0.0121008098068578" rpy="0 0 0"/>
-            <!-- <mass value="0.486218814966626"/> -->
-            <mass value="2.415"/> <!--corrected mass value measured w/o wheels-->
+            <origin xyz = '0.00498197982182523 5.70233829969297E-05 -0.0121008098068578' rpy = '0 0 0'/>
+            <mass value = '2.415'/> <!--corrected mass value measured without wheels-->
             <inertia
-                    ixx="${a*0.00196277727666921}"
-                    ixy="${a*2.50447049446755E-07}"
-                    ixz="${a*0.000140534767811098}"
-                    iyy="${a*0.00457256033711368}"
-                    iyz="${a*2.68618064993882E-07}"
-                    izz="${a*0.00493927269870476}"/>
+                    ixx = '${a*0.00196277727666921}'
+                    ixy = '${a*2.50447049446755E-07}'
+                    ixz = '${a*0.000140534767811098}'
+                    iyy = '${a*0.00457256033711368}'
+                    iyz = '${a*2.68618064993882E-07}'
+                    izz = '${a*0.00493927269870476}'/>
         </inertial>
     </link>
@@ -50,8 +50,133 @@
     </joint>
     <!-- imu to chassis joint -->
-    <joint name="base_imu" type="fixed">
-        <parent link="chassis_link"/>
-        <child link="imu_link"/>
-        <origin xyz="-0.06 0.01 0.01" rpy="0 3.1415 1.5707"/>
+    <joint name = 'base_imu' type = 'fixed'>
+        <parent link = 'chassis_link'/>
+        <child link = 'imu_link'/>
+        <origin xyz = '-0.06 0.01 0.01' rpy = '0 3.1415 1.5707'/>
+    </joint>
+    <!--WHEEL LINKS & JOINTS-->
+    <link name = 'front_right_wheel_link'>
+        <visual>
+            <origin xyz = '0 0 0' rpy = '0 0 0'/>
+            <geometry>
+                <mesh filename = 'file://$(find sim_robot_description)/meshes/front_right_wheel.STL'/>
+            </geometry>
+            <material name = 'green'/>
+        </visual>
+        <collision>
+            <origin xyz = '0 0 0' rpy = '0 0 0'/>
+            <geometry>
+                <mesh filename = 'file://$(find sim_robot_description)/meshes/front_right_wheel.STL'/>
+            </geometry>
+        </collision>
+        <inertial>
+            <origin xyz = '1.9051E-06 -2.3183E-07 -0.00064079' rpy = '0 0 0'/>
+            <mass value = '0.051532'/>
+            <inertia ixx = '${a*1.4595E-05}'
+                     ixy = '${a*-4.3975E-10}'
+                     ixz = '${a*4.415E-10}'
+                     iyy = '${a*1.4594E-05}'
+                     iyz = '${a*-1.7476E-09}'
+                     izz = '${a*2.4264E-05}'/>
+        </inertial>
+    </link>
+    <joint name = 'front_right_joint' type = 'continuous'>
+        <origin xyz = '0.08 -0.0845 -0.0389' rpy = '-1.5703 0 3.14159'/>
+        <parent link = 'chassis_link'/>
+        <child link = 'front_right_wheel_link'/>
+        <axis xyz = '0 0 1' rpy = '0 0 0'/>
+    </joint>
+    <link name = 'front_left_wheel_link'>
+        <visual>
+            <origin xyz = '0 0 0' rpy = '0 0 0'/>
+            <geometry>
+                <mesh filename = 'file://$(find sim_robot_description)/meshes/front_left_wheel.STL'/>
+            </geometry>
+            <material name = 'green'/>
+        </visual>
+        <collision>
+            <origin xyz = '0 0 0' rpy = '0 0 0'/>
+            <geometry>
+                <mesh filename = 'file://$(find sim_robot_description)/meshes/front_left_wheel.STL'/>
+            </geometry>
+        </collision>
+        <inertial>
+            <origin xyz = '2.3728E-06 -9.4228E-07 0.00064068' rpy = '0 0 0'/>
+            <mass value = '0.051543'/>
+            <inertia ixx = '${a*1.4597E-05}'
+                     ixy = '${a*-4.7945E-10}'
+                     ixz = '${a*-2.4786E-10}'
+                     iyy = '${a*1.4598E-05}'
+                     iyz = '${a*1.7972E-09}'
+                     izz = '${a*2.4267E-05}'/>
+        </inertial>
+    </link>
+    <joint name = 'front_left_joint' type = 'continuous'>
+        <origin xyz = '0.08 0.084492 -0.0389' rpy = '1.5703 0 0'/>
+        <parent link = 'chassis_link'/>
+        <child link = 'front_left_wheel_link'/>
+        <axis xyz = '0 0 1' rpy = '0 0 0'/>
+    </joint>
+    <link name = 'back_right_wheel_link'>
+        <visual>
+            <origin xyz = '0 0 0' rpy = '0 0 0'/>
+            <geometry>
+                <mesh filename = 'file://$(find sim_robot_description)/meshes/back_right_wheel.STL'/>
+            </geometry>
+            <material name = 'green'/>
+        </visual>
+        <collision>
+            <origin xyz = '0 0 0' rpy = '0 0 0'/>
+            <geometry>
+                <mesh filename = 'file://$(find sim_robot_description)/meshes/back_right_wheel.STL'/>
+            </geometry>
+        </collision>
+        <inertial>
+            <origin xyz = '-1.75924169923403E-06 1.28388821071107E-06 -0.000590549296238266' rpy = '0 0 0'/>
+            <mass value = '0.051540174053366'/>
+            <inertia ixx = '${a*1.45974152250002E-05}'
+                     ixy = '${a*1.94850559178397E-10}'
+                     ixz = '${a*-1.61846387282284E-09}'
+                     iyy = '${a*1.4596501955693E-05}'
+                     iyz = '${a*-6.27904057423818E-10}'
+                     izz = '${a*2.42663091380451E-05}'/>
+        </inertial>
+    </link>
+    <joint name = 'back_right_joint' type = 'continuous'>
+        <origin xyz = '-0.08 -0.0845 -0.03946' rpy = '-1.57 0 3.14159'/>
+        <parent link = 'chassis_link'/>
+        <child link = 'back_right_wheel_link'/>
+        <axis xyz = '0 0 1' rpy = '0 0 0'/>
+    </joint>
+    <link name = 'back_left_wheel_link'>
+        <visual>
+            <origin xyz = '0 0 0' rpy = '0 0 0'/>
+            <geometry>
+                <mesh filename = 'file://$(find sim_robot_description)/meshes/back_left_wheel.STL'/>
+            </geometry>
+            <material name = 'green'/>
+        </visual>
+        <collision>
+            <origin xyz = '0 0 0' rpy = '0 0 0'/>
+            <geometry>
+                <mesh filename = 'file://$(find sim_robot_description)/meshes/back_left_wheel.STL'/>
+            </geometry>
+        </collision>
+        <inertial>
+            <origin xyz = '-4.01213085227115E-07 2.04910264598596E-06 0.000590775697051377' rpy = '0 0 0'/>
+            <mass value = '0.0515309299357028'/>
+            <inertia ixx = '${a*1.45942986129926E-05}'
+                     ixy = '${a*-3.19787215398093E-10}'
+                     ixz = '${a*1.74943062058915E-09}'
+                     iyy = '${a*1.45948727598913E-05}'
+                     iyz = '${a*1.61769812110049E-10}'
+                     izz = '${a*2.4263683888153E-05}'/>
+        </inertial>
+    </link>
+    <joint name = 'back_left_joint' type = 'continuous'>
+        <origin xyz = '-0.08 0.084492 -0.03954' rpy = '1.5703 0 0'/>
+        <parent link = 'chassis_link'/>
+        <child link = 'back_left_wheel_link'/>
+        <axis xyz = '0 0 1' rpy = '0 0 0'/>
     </joint>
 </robot>

Commit message: tidied URDF a bit more, commented sections and adding joint damping

File: sim_robot_description/urdf/robot_body.xacro (robot description, xacro)
@@ -2,5 +2,6 @@
 <robot xmlns:xacro = 'http://www.ros.org/wiki/xacro'>
     <!-- PROPERTIES -->
-    <xacro:property name='a' value='4'/>
+    <xacro:property name = 'a' value = '4'/>    <!--scalar used for inertia -->
+    <xacro:property name = 'd' value = '0.5'/>  <!--scalar used for damping -->
     <material name = 'black'>
         <color rgba = '0.1 0.1 0.1 1'/>
@@ -9,5 +10,5 @@
         <color rgba = '0 0.7 0 1'/>
     </material>
-    <!-- BASE LINK & JOINTS-->
+    <!--            BASE LINK & JOINTS           -->
     <!-- base link -->
     <link name = 'base_link'>
@@ -55,5 +56,6 @@
         <origin xyz = '-0.06 0.01 0.01' rpy = '0 3.1415 1.5707'/>
     </joint>
-    <!--WHEEL LINKS & JOINTS-->
+    <!--            WHEEL LINKS & JOINTS             -->
+    <!-- front right wheel link -->
     <link name = 'front_right_wheel_link'>
         <visual>
@@ -81,4 +83,5 @@
         </inertial>
     </link>
+    <!-- front right wheel to chassis joint -->
     <joint name = 'front_right_joint' type = 'continuous'>
         <origin xyz = '0.08 -0.0845 -0.0389' rpy = '-1.5703 0 3.14159'/>
@@ -86,5 +89,7 @@
         <child link = 'front_right_wheel_link'/>
         <axis xyz = '0 0 1' rpy = '0 0 0'/>
+        <dynamics damping = '${d}'/>
     </joint>
+    <!-- front left wheel link -->
     <link name = 'front_left_wheel_link'>
         <visual>
@@ -112,4 +117,5 @@
         </inertial>
     </link>
+    <!-- front left wheel to chassis joint -->
     <joint name = 'front_left_joint' type = 'continuous'>
         <origin xyz = '0.08 0.084492 -0.0389' rpy = '1.5703 0 0'/>
@@ -117,5 +123,7 @@
         <child link = 'front_left_wheel_link'/>
         <axis xyz = '0 0 1' rpy = '0 0 0'/>
+        <dynamics damping = '${d}'/>
     </joint>
+    <!-- back right wheel link -->
     <link name = 'back_right_wheel_link'>
         <visual>
@@ -143,4 +151,5 @@
         </inertial>
     </link>
+    <!-- back right wheel to chassis joint -->
     <joint name = 'back_right_joint' type = 'continuous'>
         <origin xyz = '-0.08 -0.0845 -0.03946' rpy = '-1.57 0 3.14159'/>
@@ -148,5 +157,7 @@
         <child link = 'back_right_wheel_link'/>
         <axis xyz = '0 0 1' rpy = '0 0 0'/>
+        <dynamics damping = '${d}'/>
     </joint>
+    <!-- back left wheel link -->
     <link name = 'back_left_wheel_link'>
         <visual>
@@ -174,4 +185,5 @@
         </inertial>
     </link>
+    <!-- back left wheel to chassis joint -->
     <joint name = 'back_left_joint' type = 'continuous'>
         <origin xyz = '-0.08 0.084492 -0.03954' rpy = '1.5703 0 0'/>
@@ -179,4 +191,5 @@
         <child link = 'back_left_wheel_link'/>
         <axis xyz = '0 0 1' rpy = '0 0 0'/>
+        <dynamics damping = '${d}'/>
     </joint>
 </robot>

Commit message: colour changes

File: sim_robot_description/urdf/robot_body.xacro (robot description, xacro)
@@ -9,4 +9,7 @@
     <material name = 'green'>
         <color rgba = '0 0.7 0 1'/>
+    </material>
+    <material name = 'gray'>
+        <color rgba = '0.83 0.83 0.83 1'/>
     </material>
     <!--            BASE LINK & JOINTS           -->
@@ -64,5 +67,5 @@
                 <mesh filename = 'file://$(find sim_robot_description)/meshes/front_right_wheel.STL'/>
             </geometry>
-            <material name = 'green'/>
+            <material name = 'black'/>
         </visual>
         <collision>
@@ -98,5 +101,5 @@
                 <mesh filename = 'file://$(find sim_robot_description)/meshes/front_left_wheel.STL'/>
             </geometry>
-            <material name = 'green'/>
+            <material name = 'black'/>
         </visual>
         <collision>
@@ -132,5 +135,5 @@
                 <mesh filename = 'file://$(find sim_robot_description)/meshes/back_right_wheel.STL'/>
             </geometry>
-            <material name = 'green'/>
+            <material name = 'black'/>
         </visual>
         <collision>
@@ -166,5 +169,5 @@
                 <mesh filename = 'file://$(find sim_robot_description)/meshes/back_left_wheel.STL'/>
             </geometry>
-            <material name = 'green'/>
+            <material name = 'black'/>
         </visual>
         <collision>

Commit message: removed inertia origins

File: sim_robot_description/urdf/robot_body.xacro (robot description, xacro)
@@ -36,5 +36,4 @@
         </collision>
         <inertial>
-            <origin xyz = '0.00498197982182523 5.70233829969297E-05 -0.0121008098068578' rpy = '0 0 0'/>
             <mass value = '2.415'/> <!--corrected mass value measured without wheels-->
             <inertia
@@ -76,5 +75,4 @@
         </collision>
         <inertial>
-            <origin xyz = '1.9051E-06 -2.3183E-07 -0.00064079' rpy = '0 0 0'/>
             <mass value = '0.051532'/>
             <inertia ixx = '${a*1.4595E-05}'
@@ -110,5 +108,4 @@
         </collision>
         <inertial>
-            <origin xyz = '2.3728E-06 -9.4228E-07 0.00064068' rpy = '0 0 0'/>
             <mass value = '0.051543'/>
             <inertia ixx = '${a*1.4597E-05}'
@@ -144,5 +141,4 @@
         </collision>
         <inertial>
-            <origin xyz = '-1.75924169923403E-06 1.28388821071107E-06 -0.000590549296238266' rpy = '0 0 0'/>
             <mass value = '0.051540174053366'/>
             <inertia ixx = '${a*1.45974152250002E-05}'
@@ -178,5 +174,4 @@
         </collision>
         <inertial>
-            <origin xyz = '-4.01213085227115E-07 2.04910264598596E-06 0.000590775697051377' rpy = '0 0 0'/>
             <mass value = '0.0515309299357028'/>
             <inertia ixx = '${a*1.45942986129926E-05}'

Commit message: fixed wheel directions

File: sim_robot_description/urdf/robot_body.xacro (robot description, xacro)
@@ -89,5 +89,5 @@
         <parent link = 'chassis_link'/>
         <child link = 'front_right_wheel_link'/>
-        <axis xyz = '0 0 1' rpy = '0 0 0'/>
+        <axis xyz = '0 0 -1' rpy = '0 0 0'/>
         <dynamics damping = '${d}'/>
     </joint>
@@ -122,5 +122,5 @@
         <parent link = 'chassis_link'/>
         <child link = 'front_left_wheel_link'/>
-        <axis xyz = '0 0 1' rpy = '0 0 0'/>
+        <axis xyz = '0 0 -1' rpy = '0 0 0'/>
         <dynamics damping = '${d}'/>
     </joint>
@@ -155,5 +155,5 @@
         <parent link = 'chassis_link'/>
         <child link = 'back_right_wheel_link'/>
-        <axis xyz = '0 0 1' rpy = '0 0 0'/>
+        <axis xyz = '0 0 -1' rpy = '0 0 0'/>
         <dynamics damping = '${d}'/>
     </joint>
@@ -188,5 +188,5 @@
         <parent link = 'chassis_link'/>
         <child link = 'back_left_wheel_link'/>
-        <axis xyz = '0 0 1' rpy = '0 0 0'/>
+        <axis xyz = '0 0 -1' rpy = '0 0 0'/>
         <dynamics damping = '${d}'/>
     </joint>

Commit message: simplified wheel collision to basic primitive

File: sim_robot_description/urdf/robot_body.xacro (robot description, xacro)
@@ -71,5 +71,5 @@
             <origin xyz = '0 0 0' rpy = '0 0 0'/>
             <geometry>
-                <mesh filename = 'file://$(find sim_robot_description)/meshes/front_right_wheel.STL'/>
+                <cylinder radius = '0.03115' length = '0.03035'/>
             </geometry>
         </collision>
@@ -104,5 +104,5 @@
             <origin xyz = '0 0 0' rpy = '0 0 0'/>
             <geometry>
-                <mesh filename = 'file://$(find sim_robot_description)/meshes/front_left_wheel.STL'/>
+                <cylinder radius = '0.03115' length = '0.03035'/>
             </geometry>
         </collision>
@@ -137,5 +137,5 @@
             <origin xyz = '0 0 0' rpy = '0 0 0'/>
             <geometry>
-                <mesh filename = 'file://$(find sim_robot_description)/meshes/back_right_wheel.STL'/>
+                <cylinder radius = '0.03115' length = '0.03035'/>
             </geometry>
         </collision>
@@ -170,5 +170,5 @@
             <origin xyz = '0 0 0' rpy = '0 0 0'/>
             <geometry>
-                <mesh filename = 'file://$(find sim_robot_description)/meshes/back_left_wheel.STL'/>
+                <cylinder radius = '0.03115' length = '0.03035'/>
             </geometry>
         </collision>

Commit message: still can't get mecanum movement to work correctly, should follow video I found

File: sim_robot_description/urdf/robot_body.xacro (robot description, xacro)
@@ -3,5 +3,5 @@
     <!-- PROPERTIES -->
     <xacro:property name = 'a' value = '1.0'/>      <!-- scalar used for inertia -->
-    <xacro:property name = 'd' value = '0.3'/>      <!-- scalar used for damping -->
+    <xacro:property name = 'd' value = '0.1'/>     <!-- scalar used for damping -->
     <xacro:property name = 'o' value = '0.000'/>    <!-- tuneable offset for wheel collision -->
     <material name = 'black'>
@@ -84,4 +84,5 @@
             <geometry>
                 <cylinder radius = '0.0325' length = '0.03035'/>
+                <!-- <sphere radius = '0.0325'/> -->
             </geometry>
         </collision>
@@ -97,5 +98,5 @@
     <!-- front right wheel to chassis joint -->
     <joint name = 'front_right_joint' type = 'continuous'>
-        <origin xyz = '0.08 -0.0845 -0.0389' rpy = '-1.5703 0 3.14159'/>
+        <origin xyz = '0.08 -0.08475 -0.0389' rpy = '-1.5703 0 3.14159'/>
         <parent link = 'chassis_link'/>
         <child link = 'front_right_wheel_link'/>
@@ -116,4 +117,5 @@
             <geometry>
                 <cylinder radius = '0.0325' length = '0.03035'/>
+                <!-- <sphere radius = '0.0325'/> -->
             </geometry>
         </collision>
@@ -129,5 +131,5 @@
     <!-- front left wheel to chassis joint -->
     <joint name = 'front_left_joint' type = 'continuous'>
-        <origin xyz = '0.08 0.084492 -0.0389' rpy = '1.5703 0 0'/>
+        <origin xyz = '0.08 0.08475 -0.0389' rpy = '1.5703 0 0'/>
         <parent link = 'chassis_link'/>
         <child link = 'front_left_wheel_link'/>
@@ -148,4 +150,5 @@
             <geometry>
                 <cylinder radius = '0.0325' length = '0.03035'/>
+                <!-- <sphere radius = '0.0325'/> -->
             </geometry>
         </collision>
@@ -161,5 +164,5 @@
     <!-- back right wheel to chassis joint -->
     <joint name = 'back_right_joint' type = 'continuous'>
-        <origin xyz = '-0.08 -0.0845 -0.03946' rpy = '-1.57 0 3.14159'/>
+        <origin xyz = '-0.08 -0.08475 -0.03946' rpy = '-1.57 0 3.14159'/>
         <parent link = 'chassis_link'/>
         <child link = 'back_right_wheel_link'/>
@@ -180,4 +183,5 @@
             <geometry>
                 <cylinder radius = '0.0325' length = '0.03035'/>
+                <!-- <sphere radius = '0.0325'/> -->
             </geometry>
         </collision>
@@ -193,5 +197,5 @@
     <!-- back left wheel to chassis joint -->
     <joint name = 'back_left_joint' type = 'continuous'>
-        <origin xyz = '-0.08 0.084492 -0.03954' rpy = '1.5703 0 0'/>
+        <origin xyz = '-0.08 0.08475 -0.03954' rpy = '1.5703 0 0'/>
         <parent link = 'chassis_link'/>
         <child link = 'back_left_wheel_link'/>

File: sim_robot_description/urdf/robot_gazebo_properties.xacro (robot description, xacro)
@@ -2,6 +2,6 @@
 <robot xmlns:xacro="http://www.ros.org/wiki/xacro">
     <!--            PROPERTIES          -->
-    <xacro:property name = 'mu1' value = '0.7'/>
-    <xacro:property name = 'mu2' value = '0.7'/>
+    <xacro:property name = 'mu1' value = '1.5'/>
+    <xacro:property name = 'mu2' value = '0.05'/>
     <!--            LINKS          -->
     <gazebo reference = 'chassis_link'>
@@ -12,7 +12,7 @@
         <mu1 value = '${mu1}' />
         <mu2 value = '${mu2}' />
-        <minDepth>0.0001</minDepth>
-        <kp>100000</kp>
-        <kd>2500</kd>
+        <minDepth>0.001</minDepth>
+        <kp>500000</kp>
+        <kd>1</kd>
     </gazebo>
     <gazebo reference = 'front_left_wheel_link'>
@@ -20,7 +20,7 @@
         <mu1 value = '${mu1}' />
         <mu2 value = '${mu2}' />
-        <minDepth>0.0001</minDepth>
-        <kp>100000</kp>
-        <kd>2500</kd>
+        <minDepth>0.001</minDepth>
+        <kp>500000</kp>
+        <kd>1</kd>
     </gazebo>
     <gazebo reference = 'back_right_wheel_link'>
@@ -28,7 +28,7 @@
         <mu1 value = '${mu1}' />
         <mu2 value = '${mu2}' />
-        <minDepth>0.0001</minDepth>
-        <kp>100000</kp>
-        <kd>2500</kd>
+        <minDepth>0.001</minDepth>
+        <kp>500000</kp>
+        <kd>1</kd>
     </gazebo>
     <gazebo reference = 'back_left_wheel_link'>
@@ -36,7 +36,7 @@
         <mu1 value = '${mu1}' />
         <mu2 value = '${mu2}' />
-        <minDepth>0.0001</minDepth>
-        <kp>100000</kp>
-        <kd>2500</kd>
+        <minDepth>0.001</minDepth>
+        <kp>500000</kp>
+        <kd>1</kd>
     </gazebo>
     <gazebo reference = 'lidar_link'>
@@ -56,11 +56,11 @@
             <wheel_radius>0.0325</wheel_radius>
             <base_length>0.16</base_length>
-            <base_width>0.169</base_width>
+            <base_width>0.1695</base_width>
             <front_right_joint>front_right_joint</front_right_joint>
             <front_left_joint>front_left_joint</front_left_joint>
             <rear_right_joint>back_right_joint</rear_right_joint>
             <rear_left_joint>back_left_joint</rear_left_joint>
-            <wheel_max_speed>5.0</wheel_max_speed>
-            <wheel_acceleration>5.0</wheel_acceleration>
+            <wheel_max_speed>10.0</wheel_max_speed>
+            <wheel_acceleration>10.0</wheel_acceleration>
             <joint_config>1 1 1 1</joint_config>
         </plugin>
