Commit message: increased wheel mass

File: sim_robot_description/urdf/robot_body.xacro (robot description, xacro)
@@ -3,6 +3,6 @@
     <!-- PROPERTIES -->
     <xacro:property name = 'a' value = '1.0'/>      <!-- scalar used for inertia -->
-    <xacro:property name = 'd' value = '0.1'/>     <!-- scalar used for damping -->
-    <xacro:property name = 'o' value = '0.000'/>    <!-- tuneable offset for wheel collision -->
+    <xacro:property name = 'd' value = '0.0'/>     <!-- scalar used for damping -->
+    <xacro:property name = 'o' value = '0.0'/>    <!-- tuneable offset for wheel collision -->
     <material name = 'black'>
         <color rgba = '0.1 0.1 0.1 1'/>
@@ -55,5 +55,5 @@
         </collision>
         <inertial>
-            <mass value = '2.415'/>
+            <mass value = '2.415'/> <!-- mass was 2.415 -->
             <xacro:box_inertia
                 mass = '2.415'
@@ -74,5 +74,5 @@
     <link name = 'front_right_wheel_link'>
         <visual>
-            <origin xyz = '0 0 0' rpy = '0 0 0'/>
+            <origin xyz = '0 0 0' rpy = '1.5703 0 0'/>
             <geometry>
                 <mesh filename = 'file://$(find sim_robot_description)/meshes/front_right_wheel.STL'/>
@@ -81,14 +81,16 @@
         </visual>
         <collision>
-            <origin xyz = '0 ${-1 * o} 0' rpy = '0 0 0'/>
-            <geometry>
-                <cylinder radius = '0.0325' length = '0.03035'/>
-                <!-- <sphere radius = '0.0325'/> -->
-            </geometry>
-        </collision>
-        <inertial>
-            <mass value = '0.0575175'/>
-            <xacro:cylinder_inertia
-                mass = '0.0575175'
+            <origin xyz = '0 0 ${-o}' rpy = '1.5703 0 0'/>
+            <geometry>
+                <cylinder radius = '0.0325' length = '0.03035'/>
+                <!-- <sphere radius = '0.0325'/> -->
+                <!-- <mesh filename = 'file://$(find sim_robot_description)/meshes/front_right_wheel.STL'/> -->
+            </geometry>
+        </collision>
+        <inertial>
+            <!-- <mass value = '0.0575175'/> -->
+            <mass value = '10.0'/>
+            <xacro:cylinder_inertia
+                mass = '10.0'
                 radius = '0.0325'
                 length = '0.03035'
@@ -98,8 +100,8 @@
     <!-- front right wheel to chassis joint -->
     <joint name = 'front_right_joint' type = 'continuous'>
-        <origin xyz = '0.08 -0.08475 -0.0389' rpy = '-1.5703 0 3.14159'/>
+        <origin xyz = '0.08 -0.08475 -0.0389' rpy = '0 0 0'/>
         <parent link = 'chassis_link'/>
         <child link = 'front_right_wheel_link'/>
-        <axis xyz = '0 0 -1' rpy = '0 0 0'/>
+        <axis xyz = '0 1 0' rpy = '0 0 0'/>
         <dynamics damping = '${d}'/>
     </joint>
@@ -107,5 +109,5 @@
     <link name = 'front_left_wheel_link'>
         <visual>
-            <origin xyz = '0 0 0' rpy = '0 0 0'/>
+            <origin xyz = '0 0 0' rpy = '1.5703 0 0'/>
             <geometry>
                 <mesh filename = 'file://$(find sim_robot_description)/meshes/front_left_wheel.STL'/>
@@ -114,14 +116,16 @@
         </visual>
         <collision>
-            <origin xyz = '0 ${o} 0' rpy = '0 0 0'/>
-            <geometry>
-                <cylinder radius = '0.0325' length = '0.03035'/>
-                <!-- <sphere radius = '0.0325'/> -->
-            </geometry>
-        </collision>
-        <inertial>
-            <mass value = '0.0575175'/>
-            <xacro:cylinder_inertia
-                mass = '0.0575175'
+            <origin xyz = '0 0 ${-o}' rpy = '1.5703 0 0'/>
+            <geometry>
+                <cylinder radius = '0.0325' length = '0.03035'/>
+                <!-- <sphere radius = '0.0325'/> -->
+                <!-- <mesh filename = 'file://$(find sim_robot_description)/meshes/front_left_wheel.STL'/> -->
+            </geometry>
+        </collision>
+        <inertial>
+            <!-- <mass value = '0.0575175'/> -->
+            <mass value = '10.0'/>
+            <xacro:cylinder_inertia
+                mass = '10.0'
                 radius = '0.0325'
                 length = '0.03035'
@@ -131,8 +135,8 @@
     <!-- front left wheel to chassis joint -->
     <joint name = 'front_left_joint' type = 'continuous'>
-        <origin xyz = '0.08 0.08475 -0.0389' rpy = '1.5703 0 0'/>
+        <origin xyz = '0.08 0.08475 -0.0389' rpy = '0 0 0'/>
         <parent link = 'chassis_link'/>
         <child link = 'front_left_wheel_link'/>
-        <axis xyz = '0 0 -1' rpy = '0 0 0'/>
+        <axis xyz = '0 1 0' rpy = '0 0 0'/>
         <dynamics damping = '${d}'/>
     </joint>
@@ -140,5 +144,5 @@
     <link name = 'back_right_wheel_link'>
         <visual>
-            <origin xyz = '0 0 0' rpy = '0 0 0'/>
+            <origin xyz = '0 0 0' rpy = '1.5703 0 0'/>
             <geometry>
                 <mesh filename = 'file://$(find sim_robot_description)/meshes/back_right_wheel.STL'/>
@@ -147,14 +151,16 @@
         </visual>
         <collision>
-            <origin xyz = '0 ${-1 * o} 0' rpy = '0 0 0'/>
-            <geometry>
-                <cylinder radius = '0.0325' length = '0.03035'/>
-                <!-- <sphere radius = '0.0325'/> -->
-            </geometry>
-        </collision>
-        <inertial>
-            <mass value = '0.0575175'/>
-            <xacro:cylinder_inertia
-                mass = '0.0575175'
+            <origin xyz = '0 0 ${-o}' rpy = '1.5703 0 0'/>
+            <geometry>
+                <cylinder radius = '0.0325' length = '0.03035'/>
+                <!-- <sphere radius = '0.0325'/> -->
+                <!-- <mesh filename = 'file://$(find sim_robot_description)/meshes/back_right_wheel.STL'/> -->
+            </geometry>
+        </collision>
+        <inertial>
+            <!-- <mass value = '0.0575175'/> -->
+            <mass value = '10.0'/>
+            <xacro:cylinder_inertia
+                mass = '10.0'
                 radius = '0.0325'
                 length = '0.03035'
@@ -164,8 +170,8 @@
     <!-- back right wheel to chassis joint -->
     <joint name = 'back_right_joint' type = 'continuous'>
-        <origin xyz = '-0.08 -0.08475 -0.03946' rpy = '-1.57 0 3.14159'/>
+        <origin xyz = '-0.08 -0.08475 -0.0389' rpy = '0 0 0'/>   <!-- z was -0.03946 -->
         <parent link = 'chassis_link'/>
         <child link = 'back_right_wheel_link'/>
-        <axis xyz = '0 0 -1' rpy = '0 0 0'/>
+        <axis xyz = '0 1 0' rpy = '0 0 0'/>
         <dynamics damping = '${d}'/>
     </joint>
@@ -173,5 +179,5 @@
     <link name = 'back_left_wheel_link'>
         <visual>
-            <origin xyz = '0 0 0' rpy = '0 0 0'/>
+            <origin xyz = '0 0 0' rpy = '1.5703 0 0'/>
             <geometry>
                 <mesh filename = 'file://$(find sim_robot_description)/meshes/back_left_wheel.STL'/>
@@ -180,14 +186,16 @@
         </visual>
         <collision>
-            <origin xyz = '0 ${o} 0' rpy = '0 0 0'/>
-            <geometry>
-                <cylinder radius = '0.0325' length = '0.03035'/>
-                <!-- <sphere radius = '0.0325'/> -->
-            </geometry>
-        </collision>
-        <inertial>
-            <mass value = '0.0575175'/>
-            <xacro:cylinder_inertia
-                mass = '0.0575175'
+            <origin xyz = '0 0 ${-o}' rpy = '1.5703 0 0'/>
+            <geometry>
+                <cylinder radius = '0.0325' length = '0.03035'/>
+                <!-- <sphere radius = '0.0325'/> -->
+                <!-- <mesh filename = 'file://$(find sim_robot_description)/meshes/back_left_wheel.STL'/> -->
+            </geometry>
+        </collision>
+        <inertial>
+            <!-- <mass value = '0.0575175'/> -->
+            <mass value = '10.0'/>
+            <xacro:cylinder_inertia
+                mass = '10.0'
                 radius = '0.0325'
                 length = '0.03035'
@@ -197,8 +205,8 @@
     <!-- back left wheel to chassis joint -->
     <joint name = 'back_left_joint' type = 'continuous'>
-        <origin xyz = '-0.08 0.08475 -0.03954' rpy = '1.5703 0 0'/>
+        <origin xyz = '-0.08 0.08475 -0.0389' rpy = '0 0 0'/> <!-- z was -0.03954 -->
         <parent link = 'chassis_link'/>
         <child link = 'back_left_wheel_link'/>
-        <axis xyz = '0 0 -1' rpy = '0 0 0'/>
+        <axis xyz = '0 1 0' rpy = '0 0 0'/>
         <dynamics damping = '${d}'/>
     </joint>

Commit message: added mass macros

File: sim_robot_description/urdf/robot_body.xacro (robot description, xacro)
@@ -2,7 +2,9 @@
 <robot xmlns:xacro = 'http://www.ros.org/wiki/xacro'>
     <!-- PROPERTIES -->
-    <xacro:property name = 'a' value = '1.0'/>      <!-- scalar used for inertia -->
-    <xacro:property name = 'd' value = '0.0'/>     <!-- scalar used for damping -->
-    <xacro:property name = 'o' value = '0.0'/>    <!-- tuneable offset for wheel collision -->
+    <xacro:property name = 'a' value = '1.0'/>              <!-- scalar used for inertia -->
+    <xacro:property name = 'd' value = '1.0'/>              <!-- scalar used for damping -->
+    <xacro:property name = 'o' value = '0.0'/>              <!-- tuneable offset for wheel collision -->
+    <xacro:property name = 'c_mass' value = '2.415'/>       <!-- chassis mass, default is 2.415 -->
+    <xacro:property name = 'w_mass' value = '0.5'/>   <!-- wheel mass, default is 0.0575175 -->
     <material name = 'black'>
         <color rgba = '0.1 0.1 0.1 1'/>
@@ -55,7 +57,7 @@
         </collision>
         <inertial>
-            <mass value = '2.415'/> <!-- mass was 2.415 -->
+            <mass value = '${c_mass}'/>
             <xacro:box_inertia
-                mass = '2.415'
+                mass = '${c_mass}'
                 w = '0.2235'
                 h = '0.1165'
@@ -84,13 +86,10 @@
             <geometry>
                 <cylinder radius = '0.0325' length = '0.03035'/>
-                <!-- <sphere radius = '0.0325'/> -->
-                <!-- <mesh filename = 'file://$(find sim_robot_description)/meshes/front_right_wheel.STL'/> -->
-            </geometry>
-        </collision>
-        <inertial>
-            <!-- <mass value = '0.0575175'/> -->
-            <mass value = '10.0'/>
-            <xacro:cylinder_inertia
-                mass = '10.0'
+            </geometry>
+        </collision>
+        <inertial>
+            <mass value = '${w_mass}'/>
+            <xacro:cylinder_inertia
+                mass = '${w_mass}'
                 radius = '0.0325'
                 length = '0.03035'
@@ -119,13 +118,10 @@
             <geometry>
                 <cylinder radius = '0.0325' length = '0.03035'/>
-                <!-- <sphere radius = '0.0325'/> -->
-                <!-- <mesh filename = 'file://$(find sim_robot_description)/meshes/front_left_wheel.STL'/> -->
-            </geometry>
-        </collision>
-        <inertial>
-            <!-- <mass value = '0.0575175'/> -->
-            <mass value = '10.0'/>
-            <xacro:cylinder_inertia
-                mass = '10.0'
+            </geometry>
+        </collision>
+        <inertial>
+            <mass value = '${w_mass}'/>
+            <xacro:cylinder_inertia
+                mass = '${w_mass}'
                 radius = '0.0325'
                 length = '0.03035'
@@ -154,13 +150,10 @@
             <geometry>
                 <cylinder radius = '0.0325' length = '0.03035'/>
-                <!-- <sphere radius = '0.0325'/> -->
-                <!-- <mesh filename = 'file://$(find sim_robot_description)/meshes/back_right_wheel.STL'/> -->
-            </geometry>
-        </collision>
-        <inertial>
-            <!-- <mass value = '0.0575175'/> -->
-            <mass value = '10.0'/>
-            <xacro:cylinder_inertia
-                mass = '10.0'
+            </geometry>
+        </collision>
+        <inertial>
+            <mass value = '${w_mass}'/>
+            <xacro:cylinder_inertia
+                mass = '${w_mass}'
                 radius = '0.0325'
                 length = '0.03035'
@@ -189,13 +182,10 @@
             <geometry>
                 <cylinder radius = '0.0325' length = '0.03035'/>
-                <!-- <sphere radius = '0.0325'/> -->
-                <!-- <mesh filename = 'file://$(find sim_robot_description)/meshes/back_left_wheel.STL'/> -->
-            </geometry>
-        </collision>
-        <inertial>
-            <!-- <mass value = '0.0575175'/> -->
-            <mass value = '10.0'/>
-            <xacro:cylinder_inertia
-                mass = '10.0'
+            </geometry>
+        </collision>
+        <inertial>
+            <mass value = '${w_mass}'/>
+            <xacro:cylinder_inertia
+                mass = '${w_mass}'
                 radius = '0.0325'
                 length = '0.03035'

Commit message: comment change

File: sim_robot_description/urdf/robot_body.xacro (robot description, xacro)
@@ -6,5 +6,5 @@
     <xacro:property name = 'o' value = '0.0'/>              <!-- tuneable offset for wheel collision -->
     <xacro:property name = 'c_mass' value = '2.415'/>       <!-- chassis mass, default is 2.415 -->
-    <xacro:property name = 'w_mass' value = '0.5'/>   <!-- wheel mass, default is 0.0575175 -->
+    <xacro:property name = 'w_mass' value = '0.5'/>         <!-- wheel mass, default is 0.0575175 -->
     <material name = 'black'>
         <color rgba = '0.1 0.1 0.1 1'/>

Commit message: changed the wheel mass slightly

File: sim_robot_description/urdf/robot_body.xacro (robot description, xacro)
@@ -6,5 +6,5 @@
     <xacro:property name = 'o' value = '0.0'/>              <!-- tuneable offset for wheel collision -->
     <xacro:property name = 'c_mass' value = '2.415'/>       <!-- chassis mass, default is 2.415 -->
-    <xacro:property name = 'w_mass' value = '0.5'/>         <!-- wheel mass, default is 0.0575175 -->
+    <xacro:property name = 'w_mass' value = '0.575175'/>    <!-- wheel mass, default is 0.0575175 -->
     <material name = 'black'>
         <color rgba = '0.1 0.1 0.1 1'/>

Commit message: changed 'base_link' to 'base_footprint' to match odom transform

File: sim_robot_description/urdf/robot_body.xacro (robot description, xacro)
@@ -39,5 +39,5 @@
     <!-- BASE LINK & CHASSIS LINK -->
     <!-- base link -->
-    <link name = 'base_link'>
+    <link name = 'base_footprint'>
     </link>
     <!-- chassis link -->
@@ -68,5 +68,5 @@
     <!-- chassis to base joint -->
     <joint name = 'base_joint' type = 'fixed'>
-        <parent link = 'base_link'/>
+        <parent link = 'base_footprint'/>
         <child link = 'chassis_link'/>
         <origin xyz = '0 0 0.07115' rpy = '0 0 0'/> <!-- origin offset of 0.07115 -->
@@ -76,5 +76,5 @@
     <link name = 'front_right_wheel_link'>
         <visual>
-            <origin xyz = '0 0 0' rpy = '1.5703 0 0'/>
+            <origin xyz = '0 0 0' rpy = '1.570796 0 0'/>
             <geometry>
                 <mesh filename = 'file://$(find sim_robot_description)/meshes/front_right_wheel.STL'/>
@@ -83,5 +83,5 @@
         </visual>
         <collision>
-            <origin xyz = '0 0 ${-o}' rpy = '1.5703 0 0'/>
+            <origin xyz = '0 0 ${-o}' rpy = '1.570796 0 0'/>
             <geometry>
                 <cylinder radius = '0.0325' length = '0.03035'/>
@@ -108,5 +108,5 @@
     <link name = 'front_left_wheel_link'>
         <visual>
-            <origin xyz = '0 0 0' rpy = '1.5703 0 0'/>
+            <origin xyz = '0 0 0' rpy = '1.570796 0 0'/>
             <geometry>
                 <mesh filename = 'file://$(find sim_robot_description)/meshes/front_left_wheel.STL'/>
@@ -115,5 +115,5 @@
         </visual>
         <collision>
-            <origin xyz = '0 0 ${-o}' rpy = '1.5703 0 0'/>
+            <origin xyz = '0 0 ${-o}' rpy = '1.570796 0 0'/>
             <geometry>
                 <cylinder radius = '0.0325' length = '0.03035'/>
@@ -140,5 +140,5 @@
     <link name = 'back_right_wheel_link'>
         <visual>
-            <origin xyz = '0 0 0' rpy = '1.5703 0 0'/>
+            <origin xyz = '0 0 0' rpy = '1.570796 0 0'/>
             <geometry>
                 <mesh filename = 'file://$(find sim_robot_description)/meshes/back_right_wheel.STL'/>
@@ -147,5 +147,5 @@
         </visual>
         <collision>
-            <origin xyz = '0 0 ${-o}' rpy = '1.5703 0 0'/>
+            <origin xyz = '0 0 ${-o}' rpy = '1.570796 0 0'/>
             <geometry>
                 <cylinder radius = '0.0325' length = '0.03035'/>
@@ -172,5 +172,5 @@
     <link name = 'back_left_wheel_link'>
         <visual>
-            <origin xyz = '0 0 0' rpy = '1.5703 0 0'/>
+            <origin xyz = '0 0 0' rpy = '1.570796 0 0'/>
             <geometry>
                 <mesh filename = 'file://$(find sim_robot_description)/meshes/back_left_wheel.STL'/>
@@ -179,5 +179,5 @@
         </visual>
         <collision>
-            <origin xyz = '0 0 ${-o}' rpy = '1.5703 0 0'/>
+            <origin xyz = '0 0 ${-o}' rpy = '1.570796 0 0'/>
             <geometry>
                 <cylinder radius = '0.0325' length = '0.03035'/>

Commit message: changing things to better match nav2 naming conventions. issue with gazebo plugin overriding the wheel transforms

File: sim_robot_description/urdf/robot_body.xacro (robot description, xacro)
@@ -42,5 +42,5 @@
     </link>
     <!-- chassis link -->
-    <link name = 'chassis_link'>
+    <link name = 'base_link'>
         <visual>
             <origin xyz = '0 0 0' rpy = '0 0 0'/>
@@ -69,5 +69,5 @@
     <joint name = 'base_joint' type = 'fixed'>
         <parent link = 'base_footprint'/>
-        <child link = 'chassis_link'/>
+        <child link = 'base_link'/>
         <origin xyz = '0 0 0.07115' rpy = '0 0 0'/> <!-- origin offset of 0.07115 -->
     </joint>
@@ -100,5 +100,5 @@
     <joint name = 'front_right_joint' type = 'continuous'>
         <origin xyz = '0.08 -0.08475 -0.0389' rpy = '0 0 0'/>
-        <parent link = 'chassis_link'/>
+        <parent link = 'base_link'/>
         <child link = 'front_right_wheel_link'/>
         <axis xyz = '0 1 0' rpy = '0 0 0'/>
@@ -132,5 +132,5 @@
     <joint name = 'front_left_joint' type = 'continuous'>
         <origin xyz = '0.08 0.08475 -0.0389' rpy = '0 0 0'/>
-        <parent link = 'chassis_link'/>
+        <parent link = 'base_link'/>
         <child link = 'front_left_wheel_link'/>
         <axis xyz = '0 1 0' rpy = '0 0 0'/>
@@ -164,5 +164,5 @@
     <joint name = 'back_right_joint' type = 'continuous'>
         <origin xyz = '-0.08 -0.08475 -0.0389' rpy = '0 0 0'/>   <!-- z was -0.03946 -->
-        <parent link = 'chassis_link'/>
+        <parent link = 'base_link'/>
         <child link = 'back_right_wheel_link'/>
         <axis xyz = '0 1 0' rpy = '0 0 0'/>
@@ -196,5 +196,5 @@
     <joint name = 'back_left_joint' type = 'continuous'>
         <origin xyz = '-0.08 0.08475 -0.0389' rpy = '0 0 0'/> <!-- z was -0.03954 -->
-        <parent link = 'chassis_link'/>
+        <parent link = 'base_link'/>
         <child link = 'back_left_wheel_link'/>
         <axis xyz = '0 1 0' rpy = '0 0 0'/>

File: sim_robot_description/urdf/robot_gazebo_properties.xacro (robot description, xacro)
@@ -8,5 +8,5 @@
     <xacro:property name = 'kd' value = '7500'/>
     <!--            LINKS          -->
-    <gazebo reference = 'chassis_link'>
+    <gazebo reference = 'base_link'>
         <material>Gazebo/Green</material>
     </gazebo>
@@ -16,5 +16,5 @@
         <mu1 value = '${mu1}' />
         <mu2 value = '${mu2}' />
-        <fdir1 gz:expressed_in='base_link'>1 1 0</fdir1>
+        <fdir1 gz:expressed_in='base_footprint'>1 1 0</fdir1>
         <minDepth>${minDepth}</minDepth>
         <kp>${kp}</kp>
@@ -26,5 +26,5 @@
         <mu1 value = '${mu1}' />
         <mu2 value = '${mu2}' />
-        <fdir1 gz:expressed_in='base_link'>-1 1 0</fdir1>
+        <fdir1 gz:expressed_in='base_footprint'>-1 1 0</fdir1>
         <minDepth>${minDepth}</minDepth>
         <kp>${kp}</kp>
@@ -36,5 +36,5 @@
         <mu1 value = '${mu1}' />
         <mu2 value = '${mu2}' />
-        <fdir1 gz:expressed_in='base_link'>1 -1 0</fdir1>
+        <fdir1 gz:expressed_in='base_footprint'>1 -1 0</fdir1>
         <minDepth>${minDepth}</minDepth>
         <kp>${kp}</kp>
@@ -46,5 +46,5 @@
         <mu1 value = '${mu1}' />
         <mu2 value = '${mu2}' />
-        <fdir1 gz:expressed_in='base_link'>-1 -1 0</fdir1>
+        <fdir1 gz:expressed_in='base_footprint'>-1 -1 0</fdir1>
         <minDepth>${minDepth}</minDepth>
         <kp>${kp}</kp>
@@ -111,5 +111,5 @@
             <odometryFrame>odom</odometryFrame>
             <odometryRate>250.0</odometryRate>
-            <robotBaseFrame>base_footprint</robotBaseFrame>
+            <robotBaseFrame>base_link</robotBaseFrame>
             <wheel_radius>0.0325</wheel_radius>
             <base_length>0.16</base_length>

File: sim_robot_description/urdf/robot_peripherals.xacro (robot description, xacro)
@@ -29,5 +29,5 @@
     <joint name = 'lidar_joint' type = 'fixed'>
         <origin xyz = '0.0405 5.25826986680105E-05 0.08285' rpy = '0 0 0'/>
-        <parent link = 'chassis_link'/>
+        <parent link = 'base_link'/>
         <child link = 'lidar_link'/>
     </joint>
@@ -54,5 +54,5 @@
     <joint name = 'camera_joint' type = 'fixed'>
         <origin xyz = '0.057105 1.7948E-05 0.03755' rpy = '0 0 0'/>
-        <parent link = 'chassis_link'/>
+        <parent link = 'base_link'/>
         <child link = 'camera_link'/>
     </joint>
